File: miniHexa_PCB/miniHexa.kicad_pcb (KiCad board)
At the start: 4 copper layers, 94 x 65.9 mm, 82 parts, among them J2 12v DC, SW1 SW_Push, U1 STM32F401RETx, U3 RT8289GSP, U4 BQ25886RGE, U5 PCA9685BS, U6 AMS1117-3.3, Y2 25mhz

Commit message: mega update
Parts:
- removed R19: R, Resistor_SMD:R_0603_1608Metric
- removed R20: R, Resistor_SMD:R_0402_1005Metric
- removed R21: 10k, Resistor_SMD:R_0402_1005Metric
- removed Servo1, Servo10, Servo11, Servo12, Servo13, Servo14, Servo15, Servo16, Servo17, Servo18, Servo2, Servo3, Servo4, Servo5, Servo6, Servo7, Servo8, Servo9: Conn_01x03_Pin, Connector_JST:JST_XH_B3B-XH-AM_1x03_P2.50mm_Vertical
- added C31: 100nF, Capacitor_SMD:C_0402_1005Metric, F.Cu at (180.5, 80.5)
- added C32: 100nF, Capacitor_SMD:C_0402_1005Metric, F.Cu at (195.8, 88.2)
- added C33: 100nF, Capacitor_SMD:C_0402_1005Metric, F.Cu at (190.7, 75.5)
- added J1: FR_L, Connector_JST:JST_XH_B3B-XH-A_1x03_P2.50mm_Vertical, F.Cu at (148.0, 112.5)
- added J3: FR_R, Connector_JST:JST_XH_B3B-XH-A_1x03_P2.50mm_Vertical, F.Cu at (136.0, 112.5)
- added J4: MID_L, Connector_JST:JST_XH_B3B-XH-A_1x03_P2.50mm_Vertical, F.Cu at (136.0, 56.8)
- added J5: MID_R, Connector_JST:JST_XH_B3B-XH-A_1x03_P2.50mm_Vertical, F.Cu at (147.9, 56.8)
- added J6: BK_L, Connector_JST:JST_XH_B3B-XH-A_1x03_P2.50mm_Vertical, F.Cu at (183.2, 56.8)
- added J7: BK_R, Connector_JST:JST_XH_B3B-XH-A_1x03_P2.50mm_Vertical, F.Cu at (183.2, 112.7)
- added Q1: BC807, Package_TO_SOT_SMD:SOT-23, F.Cu at (145.8, 82.8)
- added R4: 10K, Resistor_SMD:R_0402_1005Metric, F.Cu at (145.8, 79.2)
- added R5: 10K, Resistor_SMD:R_0402_1005Metric, F.Cu at (145.2, 77.8)
- added R6: 10k, Resistor_SMD:R_0402_1005Metric, F.Cu at (151.8, 86.8)
- added R7: 0, Resistor_SMD:R_0603_1608Metric, F.Cu at (180.3, 84.0)
- added U2: SN74LVC1G125DBV, Package_TO_SOT_SMD:SOT-23-5, F.Cu at (141.4, 78.9)
- added U7: LSM6DS3, Package_LGA:LGA-14_3x2.5mm_P0.5mm_LayoutBorder3x4y, B.Cu at (166.9, 84.0)
- added U8: ST67W611M1A6UTR, pro_lib:U_QFN32L_ST67W611M1_STM-L, F.Cu at (187.9, 84.4)
- R2: value 0 -> 10k; footprint Resistor_SMD:R_0603_1608Metric -> Resistor_SMD:R_0402_1005Metric
- U5: value PCA9685BS -> SN74LVC1G126DBV; footprint Package_DFN_QFN:QFN-28-1EP_6x6mm_P0.65mm_EP4.25x4.25mm -> Package_TO_SOT_SMD:SOT-23-5
- moved R2 7.88 mm to (151.8, 84.0), turned to 90 degrees
- moved U5 6.22 mm to (149.8, 78.9), turned to 90 degrees
Connections:
- R2 pad 1: I2C_SCK -> +3.3V
- R2 pad 2: I2C_SCK -> SERVO_RX
- U1 pad 17: unconnected-(U1-PA3-Pad17) -> ST67_BOOT
- U1 pad 21: unconnected-(U1-PA5-Pad21) -> SP_CLK
- U1 pad 22: unconnected-(U1-PA6-Pad22) -> Net-(U1-PA6)
- U1 pad 23: unconnected-(U1-PA7-Pad23) -> SPI_MOSI
- U1 pad 25: CHIPEN_MIC_R -> unconnected-(U1-PC5-Pad25)
- U1 pad 26: SERVO17 -> unconnected-(U1-PB0-Pad26)
- U1 pad 27: SERVO18 -> unconnected-(U1-PB1-Pad27)
- U1 pad 33: unconnected-(U1-PB12-Pad33) -> SPI_CS
- U1 pad 37: CHIPEN_MIC_L -> ST67_RX
- U1 pad 38: unconnected-(U1-PC7-Pad38) -> ST67_TX
- U1 pad 39: unconnected-(U1-PC8-Pad39) -> SPI_RDY
- U1 pad 58: I2C_SCK -> SERVO_RX
- U1 pad 59: I2C_SDA -> SERVO_TX
- U1 pad 61: unconnected-(U1-PB8-Pad61) -> Net-(U1-PB8)
- U1 pad 62: unconnected-(U1-PB9-Pad62) -> Net-(U1-PB9)
- U5 pad 1: GND -> TX_EN
- U5 pad 2: +5V -> SERVO_RX
- U5 pad 3: SERVO15 -> GND
- U5 pad 4: SERVO14 -> SERVO_DATA
- U5 pad 5: SERVO13 -> +3.3V
Routing:
- net SERVO_DATA: track 0.00 -> 182.6 mm, vias 0 -> 2
- net GND: track 218.6 -> 109.9 mm, vias 20 -> 9
- net +3.3V: track 157.7 -> 97.2 mm
- net SERVO13: track 48.7 -> 0.00 mm
- net SERVO14: track 45.1 -> 0.00 mm
- net SERVO16: track 43.7 -> 0.00 mm
- net SERVO15: track 40.9 -> 0.00 mm
- net SERVO11: track 34.2 -> 0.00 mm
- net SERVO4: track 32.7 -> 0.00 mm
- net SERVO17: track 31.1 -> 0.00 mm
- net SERVO1: track 29.6 -> 0.00 mm
- net SERVO7: track 28.8 -> 0.00 mm
- net +5V: track 85.7 -> 57.3 mm, vias 2 -> 1
- net SERVO12: track 27.3 -> 0.00 mm
- net SERVO5: track 26.3 -> 0.00 mm
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- added copper zone on In1.Cu, net SERVO_DATA

Commit message: routed
Parts:
- C31, C32, C33: footprint Capacitor_SMD:C_0402_1005Metric -> Capacitor_SMD:C_0805_2012Metric
- moved C33 7.39 mm to (195.6, 81.0), turned to 90 degrees
- moved C32 0.55 mm to (195.6, 87.7)
- turned U7 to -90 degrees
Connections:
- U1 pad 41: unconnected-(U1-PA8-Pad41) -> CHIP_EN
- U8 pad 17: +3.3V -> CHIP_EN
Routing:
- net +3.3V: track 97.2 -> 190.2 mm, vias 4 -> 7
- net GND: track 109.9 -> 157.2 mm, vias 9 -> 25
- net CHIP_EN: track 0.00 -> 28.8 mm
- net ST67_BOOT: track 0.00 -> 15.0 mm
- net Net-(U1-PB8): track 0.00 -> 6.49 mm, vias 0 -> 1
- net Net-(U1-PB9): track 0.00 -> 6.06 mm, vias 0 -> 1
- net Net-(U1-VCAP1): track 0.00 -> 1.81 mm

Commit message: update
Parts:
- added C34: 100nF, Capacitor_SMD:C_0402_1005Metric, B.Cu at (167.0, 86.7)
- added C35: 100nF, Capacitor_SMD:C_0402_1005Metric, B.Cu at (168.9, 84.0)
- added R8: 4.7k, Resistor_SMD:R_0402_1005Metric, B.Cu at (163.2, 82.9)
- added R9: 4.7k, Resistor_SMD:R_0402_1005Metric, B.Cu at (164.9, 82.1)
- moved C17 1.90 mm to (164.7, 87.8)
- moved C18 1.90 mm to (166.0, 87.8)
Connections:
- U1 pad 40: unconnected-(U1-PC9-Pad40) -> IMU_INT1
- U7 pad 13: Net-(U1-PB9) -> Net-(U1-PB8)
- U7 pad 14: Net-(U1-PB8) -> Net-(U1-PB9)
- U7 pad 4: unconnected-(U7-INT1-Pad4) -> IMU_INT1
Routing:
- net GND: track 157.2 -> 166.2 mm, vias 25 -> 27
- net +3.3V: track 190.2 -> 195.7 mm, vias 7 -> 9
- net IMU_INT1: track 0.00 -> 4.19 mm, vias 0 -> 1
- net Net-(U1-PB9): track 6.06 -> 7.69 mm
- net Net-(U1-PB8): track 6.49 -> 7.84 mm

Commit message: updated pcb version
Parts:
- removed kibuzzard-6A883C46: G***, kibuzzard-6A883C46
- added kibuzzard-6AB37117: G***, kibuzzard-6AB37117, B.Cu at (133.6, 86.1)
- moved J6 1.50 mm to (181.8, 56.8)
- moved J7 1.50 mm to (181.8, 112.7)
Routing:
- net SERVO_DATA: track 182.6 -> 180.6 mm
