File: miniHexa_PCB/miniHexa.kicad_sch (KiCad schematic)
At the start: 33 parts, among them SW1 SW_Push, U1 STM32F401RETx, U7 LSM6DSL, U8 ST67W611M1A6UTR, Y2 25mhz

Commit message: changed footprint for pol cap; Need to adjust font size for the silk screen
Parts:
- removed JP1, JP2: 0hm, Resistor_SMD:R_0603_1608Metric, symbol Jumper:Jumper_2_Bridged
- added R3, R7: 0, Resistor_SMD:R_0603_1608Metric, symbol Device:R
Connections:
- net MIC_SCK: now also R3.2
- net SPI_MISO: now also R7.1
- net at U1.22 (PA6): now also R7.2
- net at U1.51 (PC10): now also R3.1
- no-connect marks 13 -> 3
Other:
- sheet POWER HANDLER renamed Power_handler
- moved on the sheet: C1, C34, C35, R32, R8, R9, U7
